Commit message: move and rename files and add macro parameters

File: urdf/sonar_single_beam.xacro (robot description, xacro)
@@ -1,5 +1,6 @@
 <?xml version="1.0"?>
 <robot xmlns:xacro="http://www.ros.org/wiki/xacro">
-  <xacro:macro name="sonar_single_beam" params="namespace suffix parent_link topic *origin">
+  <!-- note: a samples value less than 3 causes Ogre::AxisAlignedBox error -->
+  <xacro:macro name="sonar_single_beam" params="namespace suffix parent_link topic beam_width samples update_rate min_range max_range *origin">
     <!-- joint to Sonar link -->
     <joint name="${namespace}_sonar_single_beam${suffix}_joint" type="fixed">
@@ -23,5 +24,5 @@
       <visual name="visual">
         <geometry>
-          <mesh filename="file://$(find nps_uw_sensors)/meshes/blueview_p900/p900.dae"/>
+          <mesh filename="file://$(find nps_uw_sensors_gazebo)/models/blueview_p900/meshes/p900.dae"/>
         </geometry>
       </visual>
@@ -31,5 +32,5 @@
     <sensor type="gpu_ray" name="ray_sensor">
       <always_on>true</always_on>
-      <update_rate>15.0</update_rate>
+      <update_rate>${update_rate}</update_rate>
       <pose>0 0 0 0 0 0</pose>
       <visualize>true</visualize>
@@ -37,8 +38,15 @@
         <scan>
           <horizontal>
-            <samples>3</samples>
+            <samples>${samples}</samples>
+            <!-- samples value less than 3 causes Ogre::AxisAlignedBox error -->
+            <xacro:if value="${samples == '1'}">
+              <min_angle>0.0</min_angle>
+              <max_angle>0.0</max_angle>
+            </xacro:if>
+            <xacro:unless value="${samples == '1'}">
+              <min_angle>${-beam_width / 2.0}</min_angle>
+              <max_angle>${beam_width / 2.0}</max_angle>
+            </xacro:unless>
             <resolution>1</resolution>
-            <min_angle>-0.1</min_angle>
-            <max_angle>0.1</max_angle>
           </horizontal>
           <vertical>
@@ -50,6 +58,6 @@
         </scan>
         <range>
-          <min>0.1</min>
-          <max>10.0</max>
+          <min>${min_range}</min>
+          <max>${max_range}</max>
         </range>
       </ray>

File: urdf/sonar_single_beam_robot.xacro (robot description, xacro)
@@ -2,5 +2,5 @@
 <robot name="sonar_single_beam_robot"
        xmlns:xacro="http://www.ros.org/wiki/xacro">
-  <xacro:include filename="$(find nps_uw_sensors)/urdf/sonar_single_beam.xacro" />
+  <xacro:include filename="$(find nps_uw_sensors_gazebo)/urdf/sonar_single_beam.xacro" />
   <link name="world"/>
   <xacro:sonar_single_beam
@@ -8,5 +8,10 @@
             suffix="1"
             parent_link="world"
-            topic="sonar_single_beam">
+            topic="sonar_single_beam"
+            beam_width="0.2"
+            samples="3"
+            update_rate="15"
+            min_range="0.1"
+            max_range="7.0">
     <origin xyz="2.1 1.0 1.0" rpy="0 0 1.5709"/>
   </xacro:sonar_single_beam>
