Commit message: Updated DVL demo "robot" to use eNovus mesh and dimensions
Also updated WHOI DVL urdf files to include an "enable_water_tracking"
element in the plugin parameters.  When enabled (1), the DVL plugin
will include water tracking results (based on robot base link motion,
so it won't account for current yet) if the NPS additions to the WHOI
DSL environment are used (it will work fine with the WHOI version).

File: urdf/uuvsim_teledyne_whn_robot.xacro (robot description, xacro)
@@ -2,41 +2,41 @@
 <robot xmlns:xacro="http://www.ros.org/wiki/xacro" name="teledyne_whn">
   <xacro:include filename="$(find nps_uw_sensors_gazebo)/urdf/uuvsim_teledyne_whn.xacro"/>
-  <link name="cylinderbot_base_link"/>
-  <link name="cylinderbot_link">
+  <link name="robot_base_link"/>
+  <link name="robot_link">
     <inertial>
       <origin xyz="0 0 0" rpy="0 0 0"/>
       <mass value="200"/>
       <inertia
-        ixx="279.17" ixy="0.0" ixz="0.0"
-        iyy="279.17" iyz="0.0"
-        izz="25.0"/>
+        ixx="96.67" ixy="0.0" ixz="0.0"
+        iyy="158.17" iyz="0.0"
+        izz="146.83"/>
     </inertial>
     <visual>
       <geometry>
-        <cylinder length="4.0" radius="0.5"/>
+        <mesh filename="package://nps_uw_sensors_gazebo/meshes/eNOVUS.dae"/>
       </geometry>
-      <origin xyz="0 0 0" rpy="0 ${0.5*pi} 0"/>
+      <origin xyz="0 0 -0.4" rpy="0 0 ${0.5*pi}"/>
     </visual>
     <collision>
       <geometry>
-        <cylinder length="4.0" radius="0.5"/>
+        <box size="2.5 1.6 1.8"/>
       </geometry>
-      <origin xyz="0 0 0" rpy="0 ${0.5*pi} 0"/>
+      <origin xyz="-0.1 0 0.5" rpy="0 0 0"/>
     </collision>
   </link>
-  <gazebo reference="cylinderbot_link">
+  <gazebo reference="robot_link">
     <material>Gazebo/Green</material>
   </gazebo>
-  <joint name="cylinderbot_base_joint" type="fixed">
+  <joint name="robot_base_joint" type="fixed">
     <origin xyz="0 0 0" rpy="0 0 0"/>
-    <parent link="cylinderbot_base_link"/>
-    <child link="cylinderbot_link"/>
+    <parent link="robot_base_link"/>
+    <child link="robot_link"/>
   </joint>
-  <xacro:dvl_sensor_enu namespace="dvl" parent_link="cylinderbot_base_link">
+  <xacro:dvl_sensor_enu namespace="dvl" parent_link="robot_base_link">
     <origin xyz="1.5 0 -0.5" rpy="0 ${0.5*pi} 0"/>
   </xacro:dvl_sensor_enu>
   <!-- Turn gravity (off) for now so that the (unpowered) robot doesn't sink like
        a rock.  Can remove this once the neutral buoyancy issue (#4) is resolved -->
-  <gazebo reference="cylinderbot_link">
+  <gazebo reference="robot_link">
     <turnGravityOff>true</turnGravityOff>
   </gazebo>

File: urdf/whoi_nortek_dvl1000_300.xacro (robot description, xacro)
@@ -85,4 +85,5 @@
           <beamAzimuthDeg3>45</beamAzimuthDeg3>
           <beamAzimuthDeg4>-45</beamAzimuthDeg4>
+          <enableWaterTrack>1</enableWaterTrack>
           <pos_z_down>true</pos_z_down>
           <collide_bitmask>0x0001</collide_bitmask>

File: urdf/whoi_nortek_dvl1000_4000.xacro (robot description, xacro)
@@ -85,4 +85,5 @@
           <beamAzimuthDeg3>45</beamAzimuthDeg3>
           <beamAzimuthDeg4>-45</beamAzimuthDeg4>
+          <enableWaterTrack>1</enableWaterTrack>
           <pos_z_down>true</pos_z_down>
           <collide_bitmask>0x0001</collide_bitmask>

File: urdf/whoi_nortek_dvl500_300.xacro (robot description, xacro)
@@ -86,4 +86,5 @@
           <beamAzimuthDeg3>45</beamAzimuthDeg3>
           <beamAzimuthDeg4>-45</beamAzimuthDeg4>
+          <enableWaterTrack>1</enableWaterTrack>
           <pos_z_down>true</pos_z_down>
           <collide_bitmask>0x0001</collide_bitmask>

File: urdf/whoi_nortek_dvl500_6000.xacro (robot description, xacro)
@@ -86,4 +86,5 @@
           <beamAzimuthDeg3>45</beamAzimuthDeg3>
           <beamAzimuthDeg4>-45</beamAzimuthDeg4>
+          <enableWaterTrack>1</enableWaterTrack>
           <pos_z_down>true</pos_z_down>
           <collide_bitmask>0x0001</collide_bitmask>

File: urdf/whoi_sonardyne_syrinx600.xacro (robot description, xacro)
@@ -86,4 +86,5 @@
           <beamAzimuthDeg3>45</beamAzimuthDeg3>
           <beamAzimuthDeg4>-45</beamAzimuthDeg4>
+          <enableWaterTrack>1</enableWaterTrack>
           <pos_z_down>true</pos_z_down>
           <collide_bitmask>0x0001</collide_bitmask>

File: urdf/whoi_teledyne_explorer_1000.xacro (robot description, xacro)
@@ -86,4 +86,5 @@
           <beamAzimuthDeg3>45</beamAzimuthDeg3>
           <beamAzimuthDeg4>-45</beamAzimuthDeg4>
+          <enableWaterTrack>1</enableWaterTrack>
           <pos_z_down>true</pos_z_down>
           <collide_bitmask>0x0001</collide_bitmask>

File: urdf/whoi_teledyne_explorer_4000.xacro (robot description, xacro)
@@ -86,4 +86,5 @@
           <beamAzimuthDeg3>45</beamAzimuthDeg3>
           <beamAzimuthDeg4>-45</beamAzimuthDeg4>
+          <enableWaterTrack>1</enableWaterTrack>
           <pos_z_down>true</pos_z_down>
           <collide_bitmask>0x0001</collide_bitmask>

File: urdf/whoi_teledyne_whn.xacro (robot description, xacro)
@@ -84,4 +84,5 @@
           <beamAzimuthDeg3>45</beamAzimuthDeg3>
           <beamAzimuthDeg4>-45</beamAzimuthDeg4>
+          <enableWaterTrack>1</enableWaterTrack>
           <pos_z_down>true</pos_z_down>
           <collide_bitmask>0x0001</collide_bitmask>

File: urdf/whoi_teledyne_whn_robot.xacro (robot description, xacro)
@@ -3,34 +3,31 @@
   <xacro:include filename="$(find nps_uw_sensors_gazebo)/urdf/whoi_teledyne_whn.xacro"/>
   <!-- Simple example "UUV" (really it's just a cylinder) -->
-  <link name="cylinderbot_base_link"/>
-  <link name="cylinderbot_link">
+  <link name="robot_base_link"/>
+  <link name="robot_link">
     <inertial>
       <origin xyz="0 0 0" rpy="0 0 0"/>
       <mass value="200"/>
       <inertia
-        ixx="279.17" ixy="0.0" ixz="0.0"
-        iyy="279.17" iyz="0.0"
-        izz="25.0"/>
+        ixx="96.67" ixy="0.0" ixz="0.0"
+        iyy="158.17" iyz="0.0"
+        izz="146.83"/>
     </inertial>
     <visual>
       <geometry>
-        <cylinder length="4.0" radius="0.5"/>
+        <mesh filename="package://nps_uw_sensors_gazebo/meshes/eNOVUS.dae"/>
       </geometry>
-      <origin xyz="0 0 0" rpy="0 ${0.5*pi} 0"/>
+      <origin xyz="0 0 -0.4" rpy="0 0 ${0.5*pi}"/>
     </visual>
     <collision>
       <geometry>
-        <cylinder length="4.0" radius="0.5"/>
+        <box size="2.5 1.6 1.8"/>
       </geometry>
-      <origin xyz="0 0 0" rpy="0 ${0.5*pi} 0"/>
+      <origin xyz="-0.1 0 0.5" rpy="0 0 0"/>
     </collision>
   </link>
-  <gazebo reference="cylinderbot_link">
-    <material>Gazebo/Green</material>
-  </gazebo>
-  <joint name="cylinderbot_base_joint" type="fixed">
+  <joint name="robot_base_joint" type="fixed">
     <origin xyz="0 0 0" rpy="0 0 0"/>  <!-- X-fwd, Y-lft, Z-up (ick!) -->
-    <parent link="cylinderbot_base_link"/>
-    <child link="cylinderbot_link"/>
+    <parent link="robot_base_link"/>
+    <child link="robot_link"/>
   </joint>
   <!-- Call the macro to attach a DVL on the UUV's forward bottom -->
@@ -38,8 +35,8 @@
     name="dvl" namespace="dvl" xyz="0 0 0"
     dvl_topic="dvl" ranges_topic="ranges"
-    robot_link="cylinderbot_link" joint_xyz="1.5 0 -0.5"/>
+    robot_link="robot_link" joint_xyz="1 0 -0.4"/>
   <!-- Turn gravity (off) for now so that the (unpowered) robot doesn't sink like
        a rock.  Can remove this once the neutral buoyancy issue (#4) is resolved -->
-  <gazebo reference="cylinderbot_link">
+  <gazebo reference="robot_link">
     <turnGravityOff>true</turnGravityOff>
   </gazebo>

Commit message: Added a side-by-side visual with the 3 DVL meshes we've got so far
The model includes the Teledyne WHN, Teledyne Explorer and Nortek
DVL1000 and is launched from the command line with
"roslaunch nps_uw_sensors_gazebo whoi_dvl_static_side_by_side.launch"

Gravity is disabled so that the plugins (WHOI version) will publish
data (even though none of the DVLs is moving) without the DVLs
falling to the ground.  An RVIZ visualization is also launched
that actually provides a better lit view of the DVL meshes.

File: urdf/uuvsim_teledyne_whn_robot.xacro (robot description, xacro)
@@ -25,7 +25,4 @@
     </collision>
   </link>
-  <gazebo reference="robot_link">
-    <material>Gazebo/Green</material>
-  </gazebo>
   <joint name="robot_base_joint" type="fixed">
     <origin xyz="0 0 0" rpy="0 0 0"/>
@@ -34,5 +31,5 @@
   </joint>
   <xacro:dvl_sensor_enu namespace="dvl" parent_link="robot_base_link">
-    <origin xyz="1.5 0 -0.5" rpy="0 ${0.5*pi} 0"/>
+    <origin xyz="1 0 -0.4" rpy="0 ${0.5*pi} 0"/>
   </xacro:dvl_sensor_enu>
   <!-- Turn gravity (off) for now so that the (unpowered) robot doesn't sink like

File: urdf/whoi_nortek_dvl1000_300.xacro (robot description, xacro)
@@ -38,7 +38,7 @@
     <link name="${name}_link">
       <inertial>
-        <mass value="0.15"/>
+        <mass value="1.3"/>
         <origin xyz="0 0 0" rpy="${pi} 0 0"/>
-        <inertia ixx="0.0004338875" ixy="0" ixz="0" iyy="0.0004338875" iyz="0" izz="0.000243675"/>
+        <inertia ixx="0.003760358333333" ixy="0" ixz="0" iyy="0.003760358333333" iyz="0" izz="0.00211185"/>
       </inertial>
       <visual>
@@ -46,5 +46,5 @@
           <mesh filename="package://nps_uw_sensors_gazebo/meshes/DVL1000-4000m.dae"/>
         </geometry>
-        <origin xyz="${xyz}" rpy="0 3.141592653589793 0"/>
+        <origin xyz="${xyz}" rpy="0 ${pi} 0"/>
       </visual>
       <collision>
@@ -75,4 +75,5 @@
           <updateRateHZ>8.0</updateRateHZ>
           <gaussianNoiseBeamVel>0.005</gaussianNoiseBeamVel>
+          <gaussianNoiseBeamWtrVel>0.015</gaussianNoiseBeamWtrVel>
           <gaussianNoiseBeamRange>0.1</gaussianNoiseBeamRange>
           <minRange>0.2</minRange>

File: urdf/whoi_nortek_dvl1000_4000.xacro (robot description, xacro)
@@ -38,7 +38,7 @@
     <link name="${name}_link">
       <inertial>
-        <mass value="1.7"/>
+        <mass value="2.7"/>
         <origin xyz="0 0 0" rpy="${pi} 0 0"/>
-        <inertia ixx="0.005191091666667" ixy="0" ixz="0" iyy="0.005191091666667" iyz="0" izz="0.00276165"/>
+        <inertia ixx="0.008244675" ixy="0" ixz="0" iyy="0.008244675" iyz="0" izz="0.00438615"/>
       </inertial>
       <visual>
@@ -46,5 +46,5 @@
           <mesh filename="package://nps_uw_sensors_gazebo/meshes/DVL1000-4000m.dae"/>
         </geometry>
-        <origin xyz="${xyz}" rpy="0 3.141592653589793 0"/>
+        <origin xyz="${xyz}" rpy="0 ${pi} 0"/>
       </visual>
       <collision>
@@ -75,4 +75,5 @@
           <updateRateHZ>8.0</updateRateHZ>
           <gaussianNoiseBeamVel>0.005</gaussianNoiseBeamVel>
+          <gaussianNoiseBeamWtrVel>0.015</gaussianNoiseBeamWtrVel>
           <gaussianNoiseBeamRange>0.1</gaussianNoiseBeamRange>
           <minRange>0.2</minRange>

File: urdf/whoi_nortek_dvl500_300.xacro (robot description, xacro)
@@ -38,7 +38,7 @@
     <link name="${name}_link">
       <inertial>
-        <mass value="0.5"/>
+        <mass value="3.5"/>
         <origin xyz="0 0 0" rpy="${pi} 0 0"/>
-        <inertia ixx="0.002798166666667" ixy="0" ixz="0" iyy="0.002798166666667" iyz="0" izz="0.00216225"/>
+        <inertia ixx="0.019587166666667" ixy="0" ixz="0" iyy="0.019587166666667" iyz="0" izz="0.01513575"/>
       </inertial>
       <visual>
@@ -47,5 +47,5 @@
           <mesh filename="package://nps_uw_sensors_gazebo/meshes/DVL1000-4000m.dae"/>
         </geometry>
-        <origin xyz="${xyz}" rpy="0 3.141592653589793 0"/>
+        <origin xyz="${xyz}" rpy="0 ${pi} 0"/>
       </visual>
       <collision>
@@ -76,4 +76,5 @@
           <updateRateHZ>8.0</updateRateHZ>
           <gaussianNoiseBeamVel>0.005</gaussianNoiseBeamVel>
+          <gaussianNoiseBeamWtrVel>0.015</gaussianNoiseBeamWtrVel>
           <gaussianNoiseBeamRange>0.1</gaussianNoiseBeamRange>
           <minRange>0.3</minRange>

File: urdf/whoi_nortek_dvl500_6000.xacro (robot description, xacro)
@@ -40,5 +40,5 @@
         <mass value="3.1"/>
         <origin xyz="0 0 0" rpy="${pi} 0 0"/>
-        <inertia ixx="0.017348633333333" ixy="0" ixz="0" iyy="0.017348633333333" iyz="0" izz="0.01340595"/>
+        <inertia ixx="0.033018366666667" ixy="0" ixz="0" iyy="0.033018366666667" iyz="0" izz="0.02551455"/>
       </inertial>
       <visual>
@@ -47,5 +47,5 @@
           <mesh filename="package://nps_uw_sensors_gazebo/meshes/DVL1000-4000m.dae"/>
         </geometry>
-        <origin xyz="${xyz}" rpy="0 3.141592653589793 0"/>
+        <origin xyz="${xyz}" rpy="0 ${pi} 0"/>
       </visual>
       <collision>
@@ -76,4 +76,5 @@
           <updateRateHZ>8.0</updateRateHZ>
           <gaussianNoiseBeamVel>0.005</gaussianNoiseBeamVel>
+          <gaussianNoiseBeamWtrVel>0.015</gaussianNoiseBeamWtrVel>
           <gaussianNoiseBeamRange>0.1</gaussianNoiseBeamRange>
           <minRange>0.3</minRange>

File: urdf/whoi_sonardyne_syrinx600.xacro (robot description, xacro)
@@ -38,7 +38,7 @@
     <link name="${name}_link">
       <inertial>
-        <mass value="7.0"/>
+        <mass value="12.0"/>
         <origin xyz="0 0 0" rpy="${pi} 0 0"/>
-        <inertia ixx="0.0429856875" ixy="0" ixz="0" iyy="0.0429856875" iyz="0" izz="0.044296875"/>
+        <inertia ixx="0.07368975" ixy="0" ixz="0" iyy="0.07368975" iyz="0" izz="0.0759375"/>
       </inertial>
       <visual>
@@ -76,4 +76,5 @@
           <updateRateHZ>10.0</updateRateHZ>
           <gaussianNoiseBeamVel>0.0022</gaussianNoiseBeamVel>
+          <gaussianNoiseBeamWtrVel>0.0044</gaussianNoiseBeamWtrVel>
           <gaussianNoiseBeamRange>0.1</gaussianNoiseBeamRange>
           <minRange>0.4</minRange>

File: urdf/whoi_teledyne_explorer_1000.xacro (robot description, xacro)
@@ -38,8 +38,8 @@
     <link name="${name}_link">
       <inertial>
-        <mass value="0.8"/>
+        <mass value="4.3"/>
         <origin xyz="0 0 0" rpy="${pi} 0 0"/>
         <!-- Different mounting orientation than other DVLs -->
-        <inertia ixx="0.0015376" ixy="0" ixz="0" iyy="0.007853866666667" iyz="0" izz="0.007853866666667"/>
+        <inertia ixx="0.0082646" ixy="0" ixz="0" iyy="0.042214533333333" iyz="0" izz="0.042214533333333"/>
       </inertial>
       <visual>
@@ -47,5 +47,5 @@
           <mesh filename="package://nps_uw_sensors_gazebo/meshes/TeledyneMarineExplorer.dae"/>
         </geometry>
-        <origin xyz="${xyz}" rpy="-1.5707963267948966 0 -1.5707963267948966"/>
+        <origin xyz="${xyz}" rpy="${-0.5*pi} 0 ${-0.5*pi}"/>
       </visual>
       <collision>
@@ -54,5 +54,5 @@
           <cylinder length="0.326" radius="0.062"/>
         </geometry>
-        <origin xyz="${xyz}" rpy="0 1.5707963267948966 0"/>
+        <origin xyz="${xyz}" rpy="0 ${0.5*pi} 0"/>
       </collision>
     </link>
@@ -76,4 +76,5 @@
           <updateRateHZ>12.0</updateRateHZ>
           <gaussianNoiseBeamVel>0.018</gaussianNoiseBeamVel>
+          <gaussianNoiseBeamWtrVel>0.048</gaussianNoiseBeamWtrVel>
           <gaussianNoiseBeamRange>0.1</gaussianNoiseBeamRange>
           <minRange>0.5</minRange>

File: urdf/whoi_teledyne_explorer_4000.xacro (robot description, xacro)
@@ -38,8 +38,8 @@
     <link name="${name}_link">
       <inertial>
-        <mass value="3.3"/>
+        <mass value="8.6"/>
         <origin xyz="0 0 0" rpy="${pi} 0 0"/>
         <!-- Different mounting orientation than other DVLs -->
-        <inertia ixx="0.0084352125" ixy="0" ixz="0" iyy="0.03676000625" iyz="0" izz="0.03676000625"/>
+        <inertia ixx="0.021982675" ixy="0" ixz="0" iyy="0.095798804166667" iyz="0" izz="0.095798804166667"/>
       </inertial>
       <visual>
@@ -47,5 +47,5 @@
           <mesh filename="package://nps_uw_sensors_gazebo/meshes/TeledyneMarineExplorer.dae"/>
         </geometry>
-        <origin xyz="${xyz}" rpy="-1.5707963267948966 0 -1.5707963267948966"/>
+        <origin xyz="${xyz}" rpy="${-0.5*pi} 0 ${-0.5*pi}"/>
       </visual>
       <collision>
@@ -54,5 +54,5 @@
           <cylinder length="0.344" radius="0.0715"/>
         </geometry>
-        <origin xyz="${xyz}" rpy="0 1.5707963267948966 0"/>
+        <origin xyz="${xyz}" rpy="0 ${0.5*pi} 0"/>
       </collision>
     </link>
@@ -76,4 +76,5 @@
           <updateRateHZ>12.0</updateRateHZ>
           <gaussianNoiseBeamVel>0.019</gaussianNoiseBeamVel>
+          <gaussianNoiseBeamWtrVel>0.025</gaussianNoiseBeamWtrVel>
           <gaussianNoiseBeamRange>0.1</gaussianNoiseBeamRange>
           <minRange>0.5</minRange>

File: urdf/whoi_teledyne_whn.xacro (robot description, xacro)
@@ -38,7 +38,7 @@
     <link name="${name}_link">
       <inertial>
-        <mass value="8.8"/>
+        <mass value="15.8"/>
         <origin xyz="0 0 0" rpy="${pi} 0 0"/>
-        <inertia ixx="0.071732122" ixy="0" ixz="0" iyy="0.071732122" iyz="0" izz="0.055786544"/>
+        <inertia ixx="0.1287917645" ixy="0" ixz="0" iyy="0.1287917645" iyz="0" izz="0.100162204"/>
       </inertial>
       <visual>
@@ -74,4 +74,5 @@
           <updateRateHZ>7.0</updateRateHZ>
           <gaussianNoiseBeamVel>0.005</gaussianNoiseBeamVel>
+          <gaussianNoiseBeamWtrVel>0.0075</gaussianNoiseBeamWtrVel>
           <gaussianNoiseBeamRange>0.1</gaussianNoiseBeamRange>
           <minRange>0.7</minRange>
