Commit message: add ray topic

File: urdf/depth_camera_sonar_single_beam.xacro (robot description, xacro)
@@ -42,6 +42,8 @@
 	  <cameraInfoTopicName>image_raw/camera_info</cameraInfoTopicName>
 	  <pointCloudTopicName>point_cloud</pointCloudTopicName>
+	  <sonarPointCloudTopicName>sonar_point_cloud</sonarPointCloudTopicName>
 	  <depthImageTopicName>image_depth</depthImageTopicName>
 	  <normalsImageTopicName>image_normals</normalsImageTopicName>
+	  <rayImageTopicName>image_ray</rayImageTopicName>
 	  <depthImageCameraInfoTopicName>image_depth/camera_info</depthImageCameraInfoTopicName>
           <frameName>forward_sonar_optical_link</frameName>
@@ -56,5 +58,5 @@
         <image>
           <width>${samples}</width>
-          <height>1</height>
+          <height>${samples}</height>
           <format>R8G8B8</format>
         </image>

File: urdf/depth_camera_sonar_single_beam_robot.xacro (robot description, xacro)
@@ -4,4 +4,5 @@
   <xacro:include filename="$(find nps_uw_sensors_gazebo)/urdf/depth_camera_sonar_single_beam.xacro" />
   <link name="world"/>
+<!--
   <xacro:depth_camera_sonar_single_beam
             namespace="depth_camera_sonar_single_beam_robot"
@@ -15,4 +16,19 @@
             max_range="7.0">
     <origin xyz="2.1 1.0 1.0" rpy="0 0 1.5709"/>
+-->
+  <xacro:depth_camera_sonar_single_beam
+            namespace="depth_camera_sonar_single_beam_robot"
+            suffix="1"
+            parent_link="world"
+            topic="depth_camera_sonar_single_beam"
+            beam_width="1.6"
+            samples="3"
+            update_rate="15"
+            min_range="0.1"
+            max_range="7.0">
+<!--    <origin xyz="0.6 1.0 1.0" rpy="0 0 1.5709"/> -->
+<!--    <origin xyz="2.1 1.0 1.0" rpy="0 0 4.71249"/> -->
+<!--    <origin xyz="0.6 6.0 1.0" rpy="0 0 4.71249"/> -->
+    <origin xyz="0.6 1.0 1.0" rpy="0 0 1.39626"/>
   </xacro:depth_camera_sonar_single_beam>
 </robot>

Commit message: add code

File: urdf/depth_camera_sonar_single_beam.xacro (robot description, xacro)
@@ -1,6 +1,6 @@
 <?xml version="1.0"?>
 <robot xmlns:xacro="http://www.ros.org/wiki/xacro">
-  <!-- note: a samples value less than 3 causes Ogre::AxisAlignedBox error -->
-  <xacro:macro name="depth_camera_sonar_single_beam" params="namespace suffix parent_link topic beam_width samples update_rate min_range max_range *origin">
+  <!-- note: a ray count of less than (3,1) causes Ogre::AxisAlignedBox error -->
+  <xacro:macro name="depth_camera_sonar_single_beam" params="namespace suffix parent_link topic beam_width horiz_count vert_count update_rate min_range max_range *origin">
     <!-- joint to Sonar link -->
     <joint name="${namespace}_depth_camera_sonar_single_beam${suffix}_joint" type="fixed">
@@ -57,10 +57,6 @@
         <horizontal_fov>${beam_width}</horizontal_fov>
         <image>
-          <width>37</width>
-          <height>9</height>
-<!--
-          <width>${samples}</width>
-          <height>${samples}</height>
--->
+          <width>${horiz_count}</width>
+          <height>${vert_count}</height>
           <format>R8G8B8</format>
         </image>

File: urdf/depth_camera_sonar_single_beam_robot.xacro (robot description, xacro)
@@ -23,5 +23,6 @@
             topic="depth_camera_sonar_single_beam"
             beam_width="1.6"
-            samples="3"
+            horiz_count="37"
+            vert_count="9"
             update_rate="15"
             min_range="0.1"
