Commit message: Updated DVL models to include current profiling field (for plugin)

File: urdf/whoi_nortek_dvl1000_300.xacro (robot description, xacro)
@@ -88,4 +88,5 @@
           <beamAzimuthDeg4>-45</beamAzimuthDeg4>
           <enableWaterTrack>1</enableWaterTrack>
+          <waterTrackBins>10</waterTrackBins>
           <pos_z_down>true</pos_z_down>
           <collide_bitmask>0x0001</collide_bitmask>

File: urdf/whoi_nortek_dvl1000_4000.xacro (robot description, xacro)
@@ -87,4 +87,5 @@
           <beamAzimuthDeg4>-45</beamAzimuthDeg4>
           <enableWaterTrack>1</enableWaterTrack>
+          <waterTrackBins>10</waterTrackBins>
           <pos_z_down>true</pos_z_down>
           <collide_bitmask>0x0001</collide_bitmask>

File: urdf/whoi_nortek_dvl500_300.xacro (robot description, xacro)
@@ -88,4 +88,5 @@
           <beamAzimuthDeg4>-45</beamAzimuthDeg4>
           <enableWaterTrack>1</enableWaterTrack>
+          <waterTrackBins>10</waterTrackBins>
           <pos_z_down>true</pos_z_down>
           <collide_bitmask>0x0001</collide_bitmask>

File: urdf/whoi_nortek_dvl500_6000.xacro (robot description, xacro)
@@ -88,4 +88,5 @@
           <beamAzimuthDeg4>-45</beamAzimuthDeg4>
           <enableWaterTrack>1</enableWaterTrack>
+          <waterTrackBins>10</waterTrackBins>
           <pos_z_down>true</pos_z_down>
           <collide_bitmask>0x0001</collide_bitmask>

File: urdf/whoi_sonardyne_syrinx600.xacro (robot description, xacro)
@@ -88,4 +88,5 @@
           <beamAzimuthDeg4>-45</beamAzimuthDeg4>
           <enableWaterTrack>1</enableWaterTrack>
+          <waterTrackBins>10</waterTrackBins>
           <pos_z_down>true</pos_z_down>
           <collide_bitmask>0x0001</collide_bitmask>

File: urdf/whoi_teledyne_explorer_1000.xacro (robot description, xacro)
@@ -88,4 +88,5 @@
           <beamAzimuthDeg4>-45</beamAzimuthDeg4>
           <enableWaterTrack>1</enableWaterTrack>
+          <waterTrackBins>10</waterTrackBins>
           <pos_z_down>true</pos_z_down>
           <collide_bitmask>0x0001</collide_bitmask>

File: urdf/whoi_teledyne_explorer_4000.xacro (robot description, xacro)
@@ -88,4 +88,5 @@
           <beamAzimuthDeg4>-45</beamAzimuthDeg4>
           <enableWaterTrack>1</enableWaterTrack>
+          <waterTrackBins>10</waterTrackBins>
           <pos_z_down>true</pos_z_down>
           <collide_bitmask>0x0001</collide_bitmask>

File: urdf/whoi_teledyne_whn.xacro (robot description, xacro)
@@ -86,4 +86,5 @@
           <beamAzimuthDeg4>-45</beamAzimuthDeg4>
           <enableWaterTrack>1</enableWaterTrack>
+          <waterTrackBins>10</waterTrackBins>
           <pos_z_down>true</pos_z_down>
           <collide_bitmask>0x0001</collide_bitmask>

File: urdf/whoi_teledyne_whn_robot.xacro (robot description, xacro)
@@ -5,10 +5,11 @@
   <link name="robot_link">
     <inertial>
+      <!-- These are RexROV values to align with hydrodynamic model -->
       <origin xyz="0 0 0" rpy="0 0 0"/>
-      <mass value="200"/>
+      <mass value="1862.87"/>
       <inertia
-        ixx="96.67" ixy="0.0" ixz="0.0"
-        iyy="158.17" iyz="0.0"
-        izz="146.83"/>
+        ixx="525.39" ixy="1.44" ixz="33.41"
+        iyy="794.20" iyz="2.6"
+        izz="691.23"/>
     </inertial>
     <visual>
@@ -25,4 +26,42 @@
     </collision>
   </link>
+  <gazebo>
+    <plugin name="uuv_plugin" filename="libuuv_underwater_object_ros_plugin.so">
+      <fluid_density>1028.0</fluid_density>
+      <flow_velocity_topic>hydrodynamics/current_velocity</flow_velocity_topic>
+      <debug>0</debug>
+      <!-- Adding the hydrodynamic and hydrostatic parameters for the vehicle-->
+      <link name="robot_link">
+        <neutrally_buoyant>0</neutrally_buoyant>
+        <volume>1.83826</volume>
+        <box>
+          <width>1.6</width>
+          <length>2.5</length>
+          <height>1.6</height>
+        </box>
+        <center_of_buoyancy>0.0 0.0 0.3</center_of_buoyancy>
+        <hydrodynamic_model>
+          <type>fossen</type>
+          <!-- Added mass: see p.28 in Berg2012 -->
+          <added_mass>
+             779.79 -6.8773 -103.32  8.5426 -165.54 -7.8033
+            -6.8773    1222   51.29  409.44 -5.8488  62.726
+            -103.32   51.29  3659.9  6.1112 -386.42  10.774
+            8.5426  409.44  6.1112   534.9 -10.027  21.019
+            -165.54 -5.8488 -386.42 -10.027  842.69 -1.1162
+            -7.8033  62.726  10.775  21.019 -1.1162  224.32
+          </added_mass>
+          <!-- Linear damping: see p.31 in Berg2012 -->
+          <linear_damping>
+            -74.82 -69.48 -728.4 -268.8 -309.77 -105
+          </linear_damping>
+          <!-- Non-linear damping: see p.30 in Berg2012 -->
+          <quadratic_damping>
+            -748.22 -992.53 -1821.01 -672 -774.44 -523.27
+          </quadratic_damping>
+        </hydrodynamic_model>
+      </link>
+    </plugin>
+  </gazebo>
   <joint name="robot_base_joint" type="fixed">
     <origin xyz="0 0 0" rpy="0 0 0"/>  <!-- X-fwd, Y-lft, Z-up (ick!) -->
