Commit message: rename files

File: urdf/depth_camera_sonar.xacro (robot description, xacro)
@@ -2,12 +2,12 @@
 <robot xmlns:xacro="http://www.ros.org/wiki/xacro">
   <!-- note: a ray count of less than (3,1) causes Ogre::AxisAlignedBox error -->
-  <xacro:macro name="depth_camera_sonar_single_beam" params="namespace suffix parent_link topic beam_width horiz_count vert_count update_rate min_range max_range *origin">
+  <xacro:macro name="depth_camera_sonar" params="namespace suffix parent_link topic beam_width horiz_count vert_count update_rate min_range max_range *origin">
     <!-- joint to Sonar link -->
-    <joint name="${namespace}_depth_camera_sonar_single_beam${suffix}_joint" type="fixed">
+    <joint name="${namespace}_depth_camera_sonar${suffix}_joint" type="fixed">
       <parent link="${parent_link}" />
-      <child link="${namespace}/depth_camera_sonar_single_beam${suffix}_link" />
+      <child link="${namespace}/depth_camera_sonar${suffix}_link" />
       <xacro:insert_block name="origin" />
     </joint>
-    <link name="${namespace}/depth_camera_sonar_single_beam${suffix}_link">
+    <link name="${namespace}/depth_camera_sonar${suffix}_link">
       <inertial>
         <origin xyz="0 0 0" rpy="0 0 0"/>
@@ -28,7 +28,7 @@
       </visual>
     </link>
-  <gazebo reference="${namespace}/depth_camera_sonar_single_beam${suffix}_link">
+  <gazebo reference="${namespace}/depth_camera_sonar${suffix}_link">
     <selfCollide>false</selfCollide>
-    <sensor type="depth" name="depth_camera_sonar_single_beam_sensor">
+    <sensor type="depth" name="depth_camera_sonar_sensor">
       <always_on>true</always_on>
       <update_rate>${update_rate}</update_rate>
@@ -36,6 +36,6 @@
       <topic>${topic}</topic>
       <pose>0 0 0 0 0 0</pose>
-      <plugin name="nps_depth_camera_sonar_single_beam_plugin" filename="libnps_gazebo_ros_depth_camera_sonar_single_beam_plugin.so">
-	  <cameraName>depth_camera_sonar_single_beam_sensor_camera</cameraName>
+      <plugin name="nps_depth_camera_sonar_plugin" filename="libnps_gazebo_ros_depth_camera_sonar_single_beam_plugin.so">
+	  <cameraName>depth_camera_sonar_sensor_camera</cameraName>
 	  <!-- ROS publication topics -->
 	  <imageTopicName>image_raw</imageTopicName>

Commit message: add diagnostics

File: urdf/depth_camera_sonar.xacro (robot description, xacro)
@@ -2,5 +2,5 @@
 <robot xmlns:xacro="http://www.ros.org/wiki/xacro">
   <!-- note: a ray count of less than (3,1) causes Ogre::AxisAlignedBox error -->
-  <xacro:macro name="depth_camera_sonar" params="namespace suffix parent_link topic beam_width horiz_count vert_count update_rate min_range max_range *origin">
+  <xacro:macro name="depth_camera_sonar" params="namespace suffix parent_link topic beam_width horiz_count vert_count num_beams update_rate min_range max_range *origin">
     <!-- joint to Sonar link -->
     <joint name="${namespace}_depth_camera_sonar${suffix}_joint" type="fixed">
@@ -48,14 +48,9 @@
 	  <depthImageCameraInfoTopicName>image_depth/camera_info</depthImageCameraInfoTopicName>
           <frameName>forward_sonar_optical_link</frameName>
-<!--
-        <robotNamespace>${namespace}</robotNamespace>
-        <frameName>${namespace}/${topic}${suffix}_link</frameName>
-        <topicName>${topic}${suffix}_sonar_range</topicName>
--->
       </plugin>
       <camera>
         <horizontal_fov>${beam_width}</horizontal_fov>
         <image>
-          <width>${horiz_count}</width>
+          <width>${horiz_count * num_beams}</width>
           <height>${vert_count}</height>
           <format>R8G8B8</format>

File: urdf/depth_camera_sonar_robot.xacro (robot description, xacro)
@@ -12,4 +12,5 @@
             horiz_count="3"
             vert_count="4"
+            num_beams="16"
             update_rate="15"
             min_range="0.1"
