Commit message: transitioning from dvl to uwlidar sensor

File: urdf/uw_lidar.xacro (robot description, xacro)
@@ -27,15 +27,9 @@
   <!-- Generates an Underwater Lidar model and attaches it to a parent link
        Sensor parameters align with those in the 3D at Depth SL3 datasheet -->
-  <xacro:macro name="uw_lidar" params="namespace parent_link *origin inertial_reference_frame">
+  <xacro:macro name="uw_lidar" params="namespace parent_link *origin">
     <xacro:uw_lidar_plugin_macro
       namespace="${namespace}"
       suffix=""
-      parent_link="${parent_link}"
-      reference_frame="${inertial_reference_frame}"
-      update_rate="7"
-      topic="dvl"
-      noise_sigma="0.005"
-      noise_amplitude="0.005"
-      scale="1">
+      parent_link="${parent_link}" >
       <xacro:insert_block name="origin"/>
     </xacro:uw_lidar_plugin_macro>
@@ -202,25 +196,62 @@
   <!-- Generates the uw_lidar model and plugin -->
   <xacro:macro name="uw_lidar_plugin_macro"
-    params="namespace suffix parent_link topic scale *origin update_rate
-    reference_frame noise_sigma noise_amplitude">
-    <link name="${namespace}/dvl${suffix}_link">
-      <inertial>
-        <mass value="8.8"/>
+    params="namespace suffix parent_link *origin">
+    <link name="${namespace}/uw_lidar${suffix}_link">
+      <inertial>
+        <mass value="20.9"/>
         <origin xyz="0 0 0" rpy="0 0 0"/>
-        <inertia ixx="0.071732122" ixy="0" ixz="0" iyy="0.071732122" iyz="0" izz="0.055786544"/>
+        <inertia ixx="0.27709917" ixy="0" ixz="0" iyy="0.11521125" iyz="0" izz="0.27709917" />
       </inertial>
       <visual>
         <geometry>
-          <mesh filename="package://nps_uw_sensors_gazebo/models/whoi_teledyne_whn/meshes/WorkhorseNavigator.dae"/>
-        </geometry>
-        <origin xyz="0 0 0" rpy="0 1.5707963267948966 0"/>
+          <mesh filename="package://nps_uw_sensors_gazebo/models/3dad_sl3/mesh/3dad_sl3.dae"/>
+        </geometry>
+        <origin xyz="0 0 0.2735" rpy="0 0 0"/>
       </visual>
       <collision>
-        <geometry>
-          <cylinder length="0.2445" radius="0.1126"/>
-        </geometry>
-        <origin xyz="0 0 0" rpy="0 1.5707963267948966 0"/>
+       <geometry>
+         <cylinder length="0.355" radius="0.105" />
+       </geometry>
+       <origin xyz="0 0 0.2735" rpy="0 1.570796 1.570796"/>
       </collision>
     </link>
+    <link name="${namespace}/uw_lidar${suffix}_base_link">
+      <inertial>
+        <mass value="2"/>
+        <origin xyz="0 0 0.0375" rpy="0 0 0"/>
+        <inertia ixx="0.0017375" ixy="0" ixz="0" iyy="0.0017375" iyz="0" izz="0.0016" />
+      </inertial>
+      <visual>
+        <geometry>
+          <mesh filename="package://nps_uw_sensors_gazebo/models/3dad_sl3/mesh/3dad_sl3.dae"/>
+        </geometry>
+        <origin xyz="0 0 0.2735" rpy="0 0 0"/>
+      </visual>
+      <collision>
+       <geometry>
+         <cylinder length="0.075" radius="0.04" />
+       </geometry>
+       <origin xyz="0 0 0.2735" rpy="0 1.570796 1.570796"/>
+      </collision>
+    </link>
+    <pose>0 0 0.0375 0 0 0</pose>
+    <collision name="base_collision">
+      <geometry>
+        <cylinder>
+          <radius>.04</radius>
+          <length>.075</length>
+        </cylinder>
+      </geometry>
+    </collision>
+    <!-- The visual is mostly a copy of the collision -->
+    <visual name="base_visual">
+      <geometry>
+        <cylinder>
+          <radius>.04</radius>
+          <length>.075</length>
+        </cylinder>
+      </geometry>
+    </visual>
+   </link>
     <joint name="${namespace}/dvl${suffix}_joint" type="revolute">
       <xacro:insert_block name="origin"/>
@@ -230,43 +261,4 @@
       <axis xyz="1 0 0"/>
     </joint>
-    <xacro:dvl_single_sonar
-      namespace="${namespace}" topic="${topic}" suffix=""
-      index="0" pitch="-0.52" yaw="0.0" update_rate="${update_rate}">
-    </xacro:dvl_single_sonar>
-    <xacro:dvl_single_sonar
-      namespace="${namespace}" topic="${topic}" suffix=""
-      index="1" pitch="0" yaw="0.52" update_rate="${update_rate}">
-    </xacro:dvl_single_sonar>
-    <xacro:dvl_single_sonar
-      namespace="${namespace}" topic="${topic}" suffix=""
-      index="2" pitch="0.52" yaw="0.0" update_rate="${update_rate}">
-    </xacro:dvl_single_sonar>
-    <xacro:dvl_single_sonar
-      namespace="${namespace}" topic="${topic}" suffix=""
-      index="3" pitch="0.0" yaw="-0.52" update_rate="${update_rate}">
-    </xacro:dvl_single_sonar>
-    <gazebo>
-      <plugin filename="libuuv_gazebo_ros_dvl_plugin.so" name="libuuv_gazebo_dvl${suffix}_plugin">
-        <robot_namespace>${namespace}</robot_namespace> <!-- (string, required): ros namespace in which the messages are published -->
-        <link_name>${parent_link}</link_name> <!-- (string, required): name of the body which holds the IMU sensor -->
-        <sensor_topic>${topic}${suffix}</sensor_topic> <!-- (string): name of the sensor output topic and prefix of service names -->
-        <update_rate>${update_rate}</update_rate> <!-- Update period [s] -->
-        <noise_sigma>${noise_sigma}</noise_sigma> <!-- std dev of position estimates in x, y, z [m/s] -->
-        <noise_amplitude>${noise_amplitude}</noise_amplitude>
-        <enable_gazebo_messages>false</enable_gazebo_messages>
-        <enable_local_ned_frame>false</enable_local_ned_frame>
-        <static_reference_frame>${reference_frame}</static_reference_frame>
-        <!-- Declaring the beams -->
-        <beam_link_name_0>${namespace}/dvl_sonar0_link</beam_link_name_0>
-        <beam_link_name_1>${namespace}/dvl_sonar1_link</beam_link_name_1>
-        <beam_link_name_2>${namespace}/dvl_sonar2_link</beam_link_name_2>
-        <beam_link_name_3>${namespace}/dvl_sonar3_link</beam_link_name_3>
-        <!-- Declaring the beam output topics -->
-        <beam_topic_0>${topic}${suffix}_sonar0</beam_topic_0>
-        <beam_topic_1>${topic}${suffix}_sonar1</beam_topic_1>
-        <beam_topic_2>${topic}${suffix}_sonar2</beam_topic_2>
-        <beam_topic_3>${topic}${suffix}_sonar3</beam_topic_3>
-      </plugin>
-    </gazebo>
   </xacro:macro>
 </robot>

File: urdf/uw_lidar_robot.xacro (robot description, xacro)
@@ -30,5 +30,5 @@
     <child link="robot_link"/>
   </joint>
-  <xacro:uw_lidar namespace="dvl" parent_link="robot_base_link" inertial_reference_frame="world">
+  <xacro:uw_lidar namespace="dvl" parent_link="robot_base_link">
     <origin xyz="1 0 1.4" rpy="0 ${0.5*pi} 0"/>
   </xacro:uw_lidar>

Commit message: lidar control function nominally functional

File: urdf/uw_lidar.xacro (robot description, xacro)
@@ -200,5 +200,5 @@
       <inertial>
         <mass value="20.9"/>
-        <origin xyz="0 0 0" rpy="0 0 0"/>
+        <origin xyz="0 0 0.163" rpy="0 0 0"/>
         <inertia ixx="0.27709917" ixy="0" ixz="0" iyy="0.11521125" iyz="0" izz="0.27709917" />
       </inertial>
@@ -207,5 +207,5 @@
           <mesh filename="package://nps_uw_sensors_gazebo/models/3dad_sl3/mesh/3dad_sl3.dae"/>
         </geometry>
-        <origin xyz="0 0 0.2735" rpy="0 0 0"/>
+        <origin xyz="0 0 0.163" rpy="0 0 0"/>
       </visual>
       <collision>
@@ -213,52 +213,94 @@
          <cylinder length="0.355" radius="0.105" />
        </geometry>
-       <origin xyz="0 0 0.2735" rpy="0 1.570796 1.570796"/>
-      </collision>
-    </link>
-    <link name="${namespace}/uw_lidar${suffix}_base_link">
-      <inertial>
-        <mass value="2"/>
+       <origin xyz="0 0 0.163" rpy="0 ${0.5*pi} ${0.5*pi}"/>
+      </collision>
+    </link>
+    <link name="${namespace}/uw_lidar${suffix}_mount_tray_link">
+      <inertial>
+        <mass value="3.29"/>
+        <origin xyz="0 0 0" rpy="0 ${0.5*pi} 0"/>
+        <inertia ixx="0.01302291666" ixy="0" ixz="0" iyy="0.01302291666" iyz="0" izz="0.0041125" />
+      </inertial>
+      <visual>
+        <geometry>
+          <mesh filename="package://nps_uw_sensors_gazebo/models/3dad_sl3/mesh/uw_lidar_mount_tray.dae"/>
+        </geometry>
+        <origin xyz="0 0.034 0.163 " rpy="0 0 0"/>
+      </visual>
+      <collision>
+       <geometry>
+         <cylinder length="0.2" radius="0.05" />
+       </geometry>
+       <origin xyz="0 0 0" rpy="0 ${0.5*pi} 0"/>
+      </collision>
+    </link>
+    <link name="${namespace}/uw_lidar${suffix}_mount_swivel_link">
+      <inertial>
+        <mass value="1"/>
         <origin xyz="0 0 0.0375" rpy="0 0 0"/>
-        <inertia ixx="0.0017375" ixy="0" ixz="0" iyy="0.0017375" iyz="0" izz="0.0016" />
-      </inertial>
-      <visual>
-        <geometry>
-          <mesh filename="package://nps_uw_sensors_gazebo/models/3dad_sl3/mesh/3dad_sl3.dae"/>
-        </geometry>
-        <origin xyz="0 0 0.2735" rpy="0 0 0"/>
+        <inertia ixx="0.000975" ixy="0" ixz="0" iyy="0.000975" iyz="0" izz="0.0010125" />
+      </inertial>
+      <visual>
+        <geometry>
+          <mesh filename="package://nps_uw_sensors_gazebo/models/3dad_sl3/mesh/uw_lidar_mount_swivel.dae"/>
+        </geometry>
+        <origin xyz="0 0.034 0.255" rpy="0 0 0"/>
       </visual>
       <collision>
        <geometry>
-         <cylinder length="0.075" radius="0.04" />
+         <cylinder length="0.075" radius="0.045" />
        </geometry>
-       <origin xyz="0 0 0.2735" rpy="0 1.570796 1.570796"/>
-      </collision>
-    </link>
-    <pose>0 0 0.0375 0 0 0</pose>
-    <collision name="base_collision">
-      <geometry>
-        <cylinder>
-          <radius>.04</radius>
-          <length>.075</length>
-        </cylinder>
-      </geometry>
-    </collision>
-    <!-- The visual is mostly a copy of the collision -->
-    <visual name="base_visual">
-      <geometry>
-        <cylinder>
-          <radius>.04</radius>
-          <length>.075</length>
-        </cylinder>
-      </geometry>
-    </visual>
-   </link>
-    <joint name="${namespace}/dvl${suffix}_joint" type="revolute">
+       <origin xyz="0 0 0.0375" rpy="0 0 0"/>
+      </collision>
+    </link>
+    <link name="${namespace}/uw_lidar${suffix}_mount_base_link">
+      <inertial>
+        <mass value="2.84"/>
+        <origin xyz="0 0 0.06" rpy="0 0 0"/>
+        <inertia ixx="0.005964" ixy="0" ixz="0" iyy="0.005964" iyz="0" izz="0.005112" />
+      </inertial>
+      <visual>
+        <geometry>
+          <mesh filename="package://nps_uw_sensors_gazebo/models/3dad_sl3/mesh/uw_lidar_mount_base.dae"/>
+        </geometry>
+        <origin xyz="0 0.034 0.375 " rpy="0 0 0"/>
+      </visual>
+      <collision>
+       <geometry>
+         <cylinder length="0.12" radius="0.06" />
+       </geometry>
+       <origin xyz="0 0 0.06" rpy="0 0 0"/>
+      </collision>
+    </link>
+    <joint name="${namespace}/uw_lidar_tray_lidar_joint" type="fixed">
+      <origin xyz="0 0 0" rpy="0 0 0"/>
+      <parent link="${namespace}/uw_lidar${suffix}_mount_tray_link"/>
+      <child link="${namespace}/uw_lidar${suffix}_link"/>
+    </joint>
+    <joint name="${namespace}/uw_lidar_swivel_tray_joint" type="revolute">
+      <origin xyz="0 0 0.092" rpy="0 0 0"/>
+      <parent link="${namespace}/uw_lidar${suffix}_mount_swivel_link"/>
+      <child link="${namespace}/uw_lidar${suffix}_mount_tray_link"/>
+      <limit upper="${pi/12}" lower="-${pi/12}" effort="0" velocity="0"/>
+      <axis xyz="1 0 0"/>
+    </joint>
+    <joint name="${namespace}/uw_lidar_base_swivel_joint" type="revolute">
+      <origin xyz="0 0 0.12" rpy="0 0 0"/>
+      <parent link="${namespace}/uw_lidar${suffix}_mount_base_link"/>
+      <child link="${namespace}/uw_lidar${suffix}_mount_swivel_link"/>
+      <limit upper="${(35*pi)/36}" lower="-${(35*pi)/36}" effort="0" velocity="0"/>
+      <axis xyz="0 0 1"/>
+    </joint>
+    <joint name="${namespace}/uw_lidar_base_joint" type="fixed">
       <xacro:insert_block name="origin"/>
       <parent link="${parent_link}"/>
-      <child link="${namespace}/dvl${suffix}_link"/>
-      <limit upper="0" lower="0" effort="0" velocity="0"/>
-      <axis xyz="1 0 0"/>
-    </joint>
+      <child link="${namespace}/uw_lidar${suffix}_mount_base_link"/>
+    </joint>
+   <gazebo>
+      <plugin name="pulse_lidar_control" filename="libgazebo_ros_pulse_lidar_plugin.so" >
+        <pan_position>-1.57079632679</pan_position>
+        <tilt_position>0</tilt_position>
+      </plugin>
+    </gazebo>
   </xacro:macro>
 </robot>

File: urdf/uw_lidar_robot.xacro (robot description, xacro)
@@ -31,5 +31,5 @@
   </joint>
   <xacro:uw_lidar namespace="dvl" parent_link="robot_base_link">
-    <origin xyz="1 0 1.4" rpy="0 ${0.5*pi} 0"/>
+    <origin xyz="0.48 0 1.41" rpy="0 0 ${pi/2}"/>
   </xacro:uw_lidar>
   <!-- Turn gravity (off) for now so that the (unpowered) robot doesn't sink like

Commit message: laser functionality restored

File: urdf/uw_lidar.xacro (robot description, xacro)
@@ -22,5 +22,5 @@
         <cylinder length="${0.000001}" radius="${0.000001}"/>
       </geometry>
-      <origin xyz="0 0 0" rpy="0 ${0.5*pi} 0"/>
+      <origin xyz="0 0 0" rpy="0 0 0"/>
     </collision>
   </xacro:macro>
@@ -194,4 +194,77 @@
     </gazebo>
   </xacro:macro>
+  <!-- Generates a Lidar sensor -->
+  <xacro:macro name="uw_lidar_sensor" params="namespace suffix update_rate">
+    <link name="${namespace}/uw_lidar${suffix}_sensor_link">
+      <inertial>
+        <mass value="0.001"/>
+        <origin xyz="0 0 0" rpy="0 0 0"/>
+        <inertia ixx="0.000000017" ixy="0" ixz="0" iyy="0.000000017" iyz="0" izz="0.000000017"/>
+      </inertial>
+      <xacro:no_collision/>
+    </link>
+    <joint name="${namespace}/uw_lidar${suffix}_sensor_joint" type="fixed">
+      <origin xyz="0.014 -0.1825 0.168" rpy="0 0 -${pi/2}"/>
+      <parent link="${namespace}/uw_lidar${suffix}_link"/>
+      <child link="${namespace}/uw_lidar${suffix}_sensor_link"/>
+    </joint>
+   <gazebo reference="${namespace}/uw_lidar${suffix}_sensor_link">
+     <sensor name="uw_lidar_sensor" type="gpu_ray">
+       <pose>0 0 0 0 0 0</pose>
+       <update_rate>${update_rate}</update_rate>
+       <visualize>true</visualize>
+       <always_on>true</always_on>
+       <plugin name="pulse_lidar_sensing" filename="libgazebo_ros_velodyne_gpu_laser.so">
+           <topicName>nps_gazebo_ros_uw/pulse_lidar/points</topicName>
+           <frameName>nps_gazebo_ros_uw/pulse_lidar_link</frameName>
+           <min_intensity>0</min_intensity>
+           <min_range>1</min_range>
+           <max_range>20</max_range>
+           <gaussianNoise>0.05</gaussianNoise>
+       </plugin>
+       <ray>
+         <!-- The scan element contains the horizontal and vertical beams.-->
+         <scan>
+           <!-- The horizontal beams -->
+           <horizontal>
+             <!-- # of horizontal beams simulates a spinning beam -->
+             <samples>1450</samples>
+             <!-- Resolution is multiplied by samples to determine number of
+                  simulated beams vs interpolated beams. See:
+                  http://sdformat.org/spec?ver=1.6&elem=sensor#horizontal_resolution
+                  -->
+             <resolution>0.1</resolution>
+             <!-- Minimum angle in radians -->
+             <min_angle>-0.26179938779</min_angle>
+             <!-- Maximum angle in radians -->
+             <max_angle>0.26179938779</max_angle>
+           </horizontal>
+           <vertical>
+             <samples>1450</samples>
+             <resolution>0.1</resolution>
+             <min_angle>-0.26179938779</min_angle>
+             <max_angle>0.26179938779</max_angle>
+           </vertical>
+         </scan>
+         <!-- Range defines characteristics of an individual beam -->
+         <range>
+           <!-- Minimum distance of the beam in meters-->
+           <min>1</min>
+           <!-- Maximum distance of the beam in meters.
+                Should be between 2 and 45 meters, depending on visibility. -->
+           <max>20</max>
+           <!-- Linear resolution of each lidar ray. This _may_ refer to depth resolution. -->
+           <resolution>0.1</resolution>
+         </range>
+         <noise>
+           <!-- Use gaussian noise -->
+           <type>gaussian</type>
+           <mean>0.0</mean>
+           <stddev>0.05</stddev>
+         </noise>
+       </ray>
+     </sensor>
+   </gazebo>
+  </xacro:macro>
   <!-- Generates the uw_lidar model and plugin -->
   <xacro:macro name="uw_lidar_plugin_macro"
@@ -297,9 +370,13 @@
       <child link="${namespace}/uw_lidar${suffix}_mount_base_link"/>
     </joint>
-   <gazebo>
-      <plugin name="pulse_lidar_control" filename="libgazebo_ros_pulse_lidar_plugin.so" >
-        <pan_position>-1.57079632679</pan_position>
-        <tilt_position>0</tilt_position>
-      </plugin>
+    <xacro:uw_lidar_sensor
+      namespace="${namespace}" suffix=""
+      update_rate="40">
+    </xacro:uw_lidar_sensor>
+    <gazebo>
+       <plugin name="pulse_lidar_control" filename="libgazebo_ros_pulse_lidar_plugin.so" >
+         <pan_position>-1.57079632679</pan_position>
+         <tilt_position>0</tilt_position>
+       </plugin>
     </gazebo>
   </xacro:macro>

Commit message: fixing names

File: urdf/uw_lidar.xacro (robot description, xacro)
@@ -196,5 +196,5 @@
   <!-- Generates a Lidar sensor -->
   <xacro:macro name="uw_lidar_sensor" params="namespace suffix update_rate">
-    <link name="${namespace}/uw_lidar${suffix}_sensor_link">
+    <link name="${namespace}/uwl${suffix}_sensor_link">
       <inertial>
         <mass value="0.001"/>
@@ -204,10 +204,10 @@
       <xacro:no_collision/>
     </link>
-    <joint name="${namespace}/uw_lidar${suffix}_sensor_joint" type="fixed">
+    <joint name="${namespace}/uwl${suffix}_sensor_joint" type="fixed">
       <origin xyz="0.014 -0.1825 0.168" rpy="0 0 -${pi/2}"/>
-      <parent link="${namespace}/uw_lidar${suffix}_link"/>
-      <child link="${namespace}/uw_lidar${suffix}_sensor_link"/>
-    </joint>
-   <gazebo reference="${namespace}/uw_lidar${suffix}_sensor_link">
+      <parent link="${namespace}/uwl${suffix}_link"/>
+      <child link="${namespace}/uwl${suffix}_sensor_link"/>
+    </joint>
+   <gazebo reference="${namespace}/uwl${suffix}_sensor_link">
      <sensor name="uw_lidar_sensor" type="gpu_ray">
        <pose>0 0 0 0 0 0</pose>
@@ -270,5 +270,5 @@
   <xacro:macro name="uw_lidar_plugin_macro"
     params="namespace suffix parent_link *origin">
-    <link name="${namespace}/uw_lidar${suffix}_link">
+    <link name="${namespace}/uwl${suffix}_link">
       <inertial>
         <mass value="20.9"/>
@@ -289,5 +289,5 @@
       </collision>
     </link>
-    <link name="${namespace}/uw_lidar${suffix}_mount_tray_link">
+    <link name="${namespace}/uwl${suffix}_mount_tray_link">
       <inertial>
         <mass value="3.29"/>
@@ -308,5 +308,5 @@
       </collision>
     </link>
-    <link name="${namespace}/uw_lidar${suffix}_mount_swivel_link">
+    <link name="${namespace}/uwl${suffix}_mount_swivel_link">
       <inertial>
         <mass value="1"/>
@@ -327,5 +327,5 @@
       </collision>
     </link>
-    <link name="${namespace}/uw_lidar${suffix}_mount_base_link">
+    <link name="${namespace}/uwl${suffix}_mount_base_link">
       <inertial>
         <mass value="2.84"/>
@@ -346,27 +346,27 @@
       </collision>
     </link>
-    <joint name="${namespace}/uw_lidar_tray_lidar_joint" type="fixed">
+    <joint name="${namespace}/uwl_tray_lidar_joint" type="fixed">
       <origin xyz="0 0 0" rpy="0 0 0"/>
-      <parent link="${namespace}/uw_lidar${suffix}_mount_tray_link"/>
-      <child link="${namespace}/uw_lidar${suffix}_link"/>
-    </joint>
-    <joint name="${namespace}/uw_lidar_swivel_tray_joint" type="revolute">
+      <parent link="${namespace}/uwl${suffix}_mount_tray_link"/>
+      <child link="${namespace}/uwl${suffix}_link"/>
+    </joint>
+    <joint name="${namespace}/uwl_swivel_tray_joint" type="revolute">
       <origin xyz="0 0 0.092" rpy="0 0 0"/>
-      <parent link="${namespace}/uw_lidar${suffix}_mount_swivel_link"/>
-      <child link="${namespace}/uw_lidar${suffix}_mount_tray_link"/>
+      <parent link="${namespace}/uwl${suffix}_mount_swivel_link"/>
+      <child link="${namespace}/uwl${suffix}_mount_tray_link"/>
       <limit upper="${pi/12}" lower="-${pi/12}" effort="0" velocity="0"/>
       <axis xyz="1 0 0"/>
     </joint>
-    <joint name="${namespace}/uw_lidar_base_swivel_joint" type="revolute">
+    <joint name="${namespace}/uwl_base_swivel_joint" type="revolute">
       <origin xyz="0 0 0.12" rpy="0 0 0"/>
-      <parent link="${namespace}/uw_lidar${suffix}_mount_base_link"/>
-      <child link="${namespace}/uw_lidar${suffix}_mount_swivel_link"/>
+      <parent link="${namespace}/uwl${suffix}_mount_base_link"/>
+      <child link="${namespace}/uwl${suffix}_mount_swivel_link"/>
       <limit upper="${(35*pi)/36}" lower="-${(35*pi)/36}" effort="0" velocity="0"/>
       <axis xyz="0 0 1"/>
     </joint>
-    <joint name="${namespace}/uw_lidar_base_joint" type="fixed">
+    <joint name="${namespace}/uwl_base_joint" type="fixed">
       <xacro:insert_block name="origin"/>
       <parent link="${parent_link}"/>
-      <child link="${namespace}/uw_lidar${suffix}_mount_base_link"/>
+      <child link="${namespace}/uwl${suffix}_mount_base_link"/>
     </joint>
     <xacro:uw_lidar_sensor
@@ -376,5 +376,5 @@
     <gazebo>
        <plugin name="pulse_lidar_control" filename="libgazebo_ros_pulse_lidar_plugin.so" >
-         <pan_position>-1.57079632679</pan_position>
+         <pan_position>-${pi/2}</pan_position>
          <tilt_position>0</tilt_position>
        </plugin>

File: urdf/uw_lidar_robot.xacro (robot description, xacro)
@@ -30,5 +30,5 @@
     <child link="robot_link"/>
   </joint>
-  <xacro:uw_lidar namespace="dvl" parent_link="robot_base_link">
+  <xacro:uw_lidar namespace="uwl" parent_link="robot_base_link">
     <origin xyz="0.48 0 1.41" rpy="0 0 ${pi/2}"/>
   </xacro:uw_lidar>
@@ -38,17 +38,17 @@
     <turnGravityOff>true</turnGravityOff>
   </gazebo>
-  <gazebo reference="dvl/dvl_link">
+  <gazebo reference="uwl/uwl_link">
     <turnGravityOff>true</turnGravityOff>
   </gazebo>
-  <gazebo reference="dvl/dvl_sonar0_link">
+  <gazebo reference="uwl/uwl_mount_tray_link">
     <turnGravityOff>true</turnGravityOff>
   </gazebo>
-  <gazebo reference="dvl/dvl_sonar1_link">
+  <gazebo reference="uwl/uwl_mount_swivel_link">
     <turnGravityOff>true</turnGravityOff>
   </gazebo>
-  <gazebo reference="dvl/dvl_sonar2_link">
+  <gazebo reference="uwl/uwl_mount_base_link">
     <turnGravityOff>true</turnGravityOff>
   </gazebo>
-  <gazebo reference="dvl/dvl_sonar3_link">
+  <gazebo reference="uwl/uwl_sensor_link">
     <turnGravityOff>true</turnGravityOff>
   </gazebo>
