Commit message: minor cleanup

File: urdf/uw_lidar.xacro (robot description, xacro)
@@ -18,4 +18,10 @@
        that we do not want to collide with anything (e.g., individual DVL sonars) -->
   <xacro:macro name="no_collision">
+    <visual>
+      <geometry>
+        <cylinder length="${0.01}" radius="${0.01}"/>
+      </geometry>
+      <origin xyz="0 0 0" rpy="0 0 0"/>
+    </visual>
     <collision>
       <geometry>
@@ -27,5 +33,5 @@
   <!-- Generates an Underwater Lidar model and attaches it to a parent link
        Sensor parameters align with those in the 3D at Depth SL3 datasheet -->
-  <xacro:macro name="uw_lidar" params="namespace parent_link *origin">
+  <xacro:macro name="uwl_macro" params="namespace parent_link *origin">
     <xacro:uw_lidar_plugin_macro
       namespace="${namespace}"
@@ -215,4 +221,5 @@
        <visualize>true</visualize>
        <always_on>true</always_on>
+<!--
        <plugin name="pulse_lidar_sensing" filename="libgazebo_ros_velodyne_gpu_laser.so">
            <topicName>nps_gazebo_ros_uw/pulse_lidar/points</topicName>
@@ -223,4 +230,5 @@
            <gaussianNoise>0.05</gaussianNoise>
        </plugin>
+-->
        <ray>
          <!-- The scan element contains the horizontal and vertical beams.-->
@@ -236,13 +244,13 @@
              <resolution>0.1</resolution>
              <!-- Minimum angle in radians -->
-             <min_angle>-0.26179938779</min_angle>
+             <min_angle>${-pi/12}</min_angle>
              <!-- Maximum angle in radians -->
-             <max_angle>0.26179938779</max_angle>
+             <max_angle>${pi/12}</max_angle>
            </horizontal>
            <vertical>
              <samples>1450</samples>
              <resolution>0.1</resolution>
-             <min_angle>-0.26179938779</min_angle>
-             <max_angle>0.26179938779</max_angle>
+             <min_angle>${-pi/12}</min_angle>
+             <max_angle>${pi/12}</max_angle>
            </vertical>
          </scan>
@@ -299,5 +307,5 @@
           <mesh filename="package://nps_uw_sensors_gazebo/models/3dad_sl3/mesh/uw_lidar_mount_tray.dae"/>
         </geometry>
-        <origin xyz="0 0.034 0.163 " rpy="0 0 0"/>
+        <origin xyz="0 0.034 0.163" rpy="0 0 0"/>
       </visual>
       <collision>
@@ -337,5 +345,5 @@
           <mesh filename="package://nps_uw_sensors_gazebo/models/3dad_sl3/mesh/uw_lidar_mount_base.dae"/>
         </geometry>
-        <origin xyz="0 0.034 0.375 " rpy="0 0 0"/>
+        <origin xyz="0 0.034 0.375" rpy="0 0 0"/>
       </visual>
       <collision>
@@ -376,6 +384,7 @@
     <gazebo>
        <plugin name="pulse_lidar_control" filename="libgazebo_ros_pulse_lidar_plugin.so" >
+        <robot_namespace>${namespace}</robot_namespace> <!-- (string, required): ros namespace in which the messages are published -->
          <pan_position>-${pi/2}</pan_position>
-         <tilt_position>0</tilt_position>
+         <tilt_position>0*${pi/18}</tilt_position>
        </plugin>
     </gazebo>

Commit message: joint effort and velocity can't be set to 0!

File: urdf/uw_lidar.xacro (robot description, xacro)
@@ -363,5 +363,5 @@
       <parent link="${namespace}/uwl${suffix}_mount_swivel_link"/>
       <child link="${namespace}/uwl${suffix}_mount_tray_link"/>
-      <limit upper="${pi/12}" lower="-${pi/12}" effort="0" velocity="0"/>
+      <limit upper="${pi/12}" lower="-${pi/12}" effort="100" velocity="20"/>
       <axis xyz="1 0 0"/>
     </joint>
@@ -370,5 +370,5 @@
       <parent link="${namespace}/uwl${suffix}_mount_base_link"/>
       <child link="${namespace}/uwl${suffix}_mount_swivel_link"/>
-      <limit upper="${(35*pi)/36}" lower="-${(35*pi)/36}" effort="0" velocity="0"/>
+      <limit upper="${(35*pi)/36}" lower="-${(35*pi)/36}" effort="100" velocity="20"/>
       <axis xyz="0 0 1"/>
     </joint>

Commit message: cleanup

File: urdf/uw_lidar.xacro (robot description, xacro)
@@ -10,8 +10,5 @@
      limitations under the License.
 -->
-<!-- Xacro macros for generating Teledyne Workhorse Navigator (WHN) class URDF models
-     utilizing the uuv_simulator DVL plugin (libuuv_gazebo_ros_dvl_plugin.so)
-     Adapted from uuv_simulator version (uuv_sensor_ros_plugins/urdf/dvl_snippets.xacro)
-     to correct naming and URDF version-based errors & configure default parameters -->
+<!-- Xacro macros for generating underwater lidar URDF model -->
 <robot xmlns:xacro="http://www.ros.org/wiki/xacro">
   <!-- Generates a tiny "no-collision" cylinder for incorporation into a link
@@ -41,163 +38,4 @@
     </xacro:uw_lidar_plugin_macro>
   </xacro:macro>
-  <!-- Generates a Teledyne WHN URDF model and attaches it to a parent link
-       Sensor parameters align with those in the WHN 600 datasheet -->
-  <xacro:macro name="dvl_macro" params="namespace parent_link *origin inertial_reference_frame">
-    <xacro:dvl_plugin_macro
-      namespace="${namespace}"
-      suffix=""
-      parent_link="${parent_link}"
-      reference_frame="${inertial_reference_frame}"
-      update_rate="7"
-      topic="dvl"
-      noise_sigma="0.005"
-      noise_amplitude="0.005"
-      scale="1">
-      <xacro:insert_block name="origin"/>
-    </xacro:dvl_plugin_macro>
-  </xacro:macro>
-  <!-- Generates an ENU Teledyne WHN URDF model and attaches it to a parent link -->
-  <xacro:macro name="dvl_sensor_enu" params="namespace parent_link *origin">
-    <xacro:dvl_macro
-      namespace="${namespace}"
-      parent_link="${parent_link}"
-      inertial_reference_frame="world">
-      <xacro:insert_block name="origin"/>
-    </xacro:dvl_macro>
-  </xacro:macro>
-  <!-- Generates an NED Teledyne WHN URDF model and attaches it to a parent link -->
-  <xacro:macro name="dvl_sensor_ned" params="namespace parent_link *origin">
-    <xacro:dvl_macro
-      namespace="${namespace}"
-      parent_link="${parent_link}"
-      inertial_reference_frame="world_ned">
-      <xacro:insert_block name="origin"/>
-    </xacro:dvl_macro>
-  </xacro:macro>
-  <!-- Generates a single ranging sonar for the DVL -->
-  <xacro:macro name="dvl_single_sonar" params="namespace topic suffix index pitch yaw update_rate">
-    <link name="${namespace}/dvl${suffix}_sonar${index}_link">
-      <inertial>
-        <mass value="0.001"/>
-        <origin xyz="0 0 0" rpy="0 0 0"/>
-        <inertia ixx="0.000000017" ixy="0" ixz="0" iyy="0.000000017" iyz="0" izz="0.000000017"/>
-      </inertial>
-      <xacro:no_collision/>
-    </link>
-    <joint name="${namespace}/dvl${suffix}_sonar${index}_joint" type="revolute">
-      <origin xyz="0 0 0" rpy="0 ${pitch} ${yaw}"/>
-      <parent link="${namespace}/dvl${suffix}_link"/>
-      <child link="${namespace}/dvl${suffix}_sonar${index}_link"/>
-      <limit upper="0" lower="0" effort="0" velocity="0"/>
-      <axis xyz="1 0 0"/>
-    </joint>
-    <gazebo reference="${namespace}/dvl${suffix}_sonar${index}_link">
-      <sensor type="ray" name="dvl${suffix}_sonar${index}">
-        <pose>0 0 0 0 0 0</pose>
-        <update_rate>${update_rate}</update_rate>
-        <visualize>true</visualize>
-        <ray>
-          <scan>
-            <horizontal>
-              <samples>3</samples>
-              <resolution>1</resolution>
-              <min_angle>-0.03</min_angle>
-              <max_angle>0.03</max_angle>
-            </horizontal>
-            <vertical>
-              <samples>3</samples>
-              <resolution>1</resolution>
-              <min_angle>-0.03</min_angle>
-              <max_angle>0.03</max_angle>
-            </vertical>
-          </scan>
-          <range>
-            <min>0.7</min>
-            <max>90</max>
-            <resolution>0.01</resolution>
-          </range>
-        </ray>
-        <plugin filename="libgazebo_ros_range.so" name="dvl${suffix}_sonar${index}">
-          <gaussianNoise>0.005</gaussianNoise>
-          <alwaysOn>true</alwaysOn>
-          <updateRate>${update_rate}</updateRate>
-          <topicName>${namespace}/${topic}${suffix}_sonar${index}</topicName>
-          <frameName>${namespace}/dvl${suffix}_sonar${index}_link</frameName>
-          <fov>0.06</fov>
-          <radiation>ultrasound</radiation>
-        </plugin>
-      </sensor>
-    </gazebo>
-  </xacro:macro>
-  <!-- Generates the DVL URDF model and plugin -->
-  <xacro:macro name="dvl_plugin_macro"
-    params="namespace suffix parent_link topic scale *origin update_rate
-    reference_frame noise_sigma noise_amplitude">
-    <link name="${namespace}/dvl${suffix}_link">
-      <inertial>
-        <mass value="8.8"/>
-        <origin xyz="0 0 0" rpy="0 0 0"/>
-        <inertia ixx="0.071732122" ixy="0" ixz="0" iyy="0.071732122" iyz="0" izz="0.055786544"/>
-      </inertial>
-      <visual>
-        <geometry>
-          <mesh filename="package://nps_uw_sensors_gazebo/models/whoi_teledyne_whn/meshes/WorkhorseNavigator.dae"/>
-        </geometry>
-        <origin xyz="0 0 0" rpy="0 1.5707963267948966 0"/>
-      </visual>
-      <collision>
-        <geometry>
-          <cylinder length="0.2445" radius="0.1126"/>
-        </geometry>
-        <origin xyz="0 0 0" rpy="0 1.5707963267948966 0"/>
-      </collision>
-    </link>
-    <joint name="${namespace}/dvl${suffix}_joint" type="revolute">
-      <xacro:insert_block name="origin"/>
-      <parent link="${parent_link}"/>
-      <child link="${namespace}/dvl${suffix}_link"/>
-      <limit upper="0" lower="0" effort="0" velocity="0"/>
-      <axis xyz="1 0 0"/>
-    </joint>
-    <xacro:dvl_single_sonar
-      namespace="${namespace}" topic="${topic}" suffix=""
-      index="0" pitch="-0.52" yaw="0.0" update_rate="${update_rate}">
-    </xacro:dvl_single_sonar>
-    <xacro:dvl_single_sonar
-      namespace="${namespace}" topic="${topic}" suffix=""
-      index="1" pitch="0" yaw="0.52" update_rate="${update_rate}">
-    </xacro:dvl_single_sonar>
-    <xacro:dvl_single_sonar
-      namespace="${namespace}" topic="${topic}" suffix=""
-      index="2" pitch="0.52" yaw="0.0" update_rate="${update_rate}">
-    </xacro:dvl_single_sonar>
-    <xacro:dvl_single_sonar
-      namespace="${namespace}" topic="${topic}" suffix=""
-      index="3" pitch="0.0" yaw="-0.52" update_rate="${update_rate}">
-    </xacro:dvl_single_sonar>
-    <gazebo>
-      <plugin filename="libuuv_gazebo_ros_dvl_plugin.so" name="libuuv_gazebo_dvl${suffix}_plugin">
-        <robot_namespace>${namespace}</robot_namespace> <!-- (string, required): ros namespace in which the messages are published -->
-        <link_name>${parent_link}</link_name> <!-- (string, required): name of the body which holds the IMU sensor -->
-        <sensor_topic>${topic}${suffix}</sensor_topic> <!-- (string): name of the sensor output topic and prefix of service names -->
-        <update_rate>${update_rate}</update_rate> <!-- Update period [s] -->
-        <noise_sigma>${noise_sigma}</noise_sigma> <!-- std dev of position estimates in x, y, z [m/s] -->
-        <noise_amplitude>${noise_amplitude}</noise_amplitude>
-        <enable_gazebo_messages>false</enable_gazebo_messages>
-        <enable_local_ned_frame>false</enable_local_ned_frame>
-        <static_reference_frame>${reference_frame}</static_reference_frame>
-        <!-- Declaring the beams -->
-        <beam_link_name_0>${namespace}/dvl_sonar0_link</beam_link_name_0>
-        <beam_link_name_1>${namespace}/dvl_sonar1_link</beam_link_name_1>
-        <beam_link_name_2>${namespace}/dvl_sonar2_link</beam_link_name_2>
-        <beam_link_name_3>${namespace}/dvl_sonar3_link</beam_link_name_3>
-        <!-- Declaring the beam output topics -->
-        <beam_topic_0>${topic}${suffix}_sonar0</beam_topic_0>
-        <beam_topic_1>${topic}${suffix}_sonar1</beam_topic_1>
-        <beam_topic_2>${topic}${suffix}_sonar2</beam_topic_2>
-        <beam_topic_3>${topic}${suffix}_sonar3</beam_topic_3>
-      </plugin>
-    </gazebo>
-  </xacro:macro>
   <!-- Generates a Lidar sensor -->
   <xacro:macro name="uw_lidar_sensor" params="namespace suffix update_rate">
@@ -221,8 +59,7 @@
        <visualize>true</visualize>
        <always_on>true</always_on>
-<!--
        <plugin name="pulse_lidar_sensing" filename="libgazebo_ros_velodyne_gpu_laser.so">
-           <topicName>nps_gazebo_ros_uw/pulse_lidar/points</topicName>
-           <frameName>nps_gazebo_ros_uw/pulse_lidar_link</frameName>
+           <topicName>nps_uwl/points</topicName>
+           <frameName>nps_uwl/pulse_lidar_link</frameName>
            <min_intensity>0</min_intensity>
            <min_range>1</min_range>
@@ -230,5 +67,4 @@
            <gaussianNoise>0.05</gaussianNoise>
        </plugin>
--->
        <ray>
          <!-- The scan element contains the horizontal and vertical beams.-->
@@ -275,5 +111,5 @@
    </gazebo>
   </xacro:macro>
-  <!-- Generates the uw_lidar model and plugin -->
+  <!-- Generates the uw_lidar model with stand and motion control plugin -->
   <xacro:macro name="uw_lidar_plugin_macro"
     params="namespace suffix parent_link *origin">
@@ -363,5 +199,5 @@
       <parent link="${namespace}/uwl${suffix}_mount_swivel_link"/>
       <child link="${namespace}/uwl${suffix}_mount_tray_link"/>
-      <limit upper="${pi/12}" lower="-${pi/12}" effort="100" velocity="20"/>
+      <limit upper="${pi/12}" lower="-${pi/12}" effort="100" velocity="100"/>
       <axis xyz="1 0 0"/>
     </joint>
@@ -370,5 +206,5 @@
       <parent link="${namespace}/uwl${suffix}_mount_base_link"/>
       <child link="${namespace}/uwl${suffix}_mount_swivel_link"/>
-      <limit upper="${(35*pi)/36}" lower="-${(35*pi)/36}" effort="100" velocity="20"/>
+      <limit upper="${(35*pi)/36}" lower="-${(35*pi)/36}" effort="100" velocity="100"/>
       <axis xyz="0 0 1"/>
     </joint>
@@ -384,7 +220,7 @@
     <gazebo>
        <plugin name="pulse_lidar_control" filename="libgazebo_ros_pulse_lidar_plugin.so" >
-        <robot_namespace>${namespace}</robot_namespace> <!-- (string, required): ros namespace in which the messages are published -->
-         <pan_position>-${pi/2}</pan_position>
-         <tilt_position>0*${pi/18}</tilt_position>
+        <robot_namespace>${namespace}</robot_namespace>
+         <pan_position>0</pan_position>
+         <tilt_position>0</tilt_position>
        </plugin>
     </gazebo>

Commit message: making initial pan and tilt configurable from uwl_macro

File: urdf/uw_lidar.xacro (robot description, xacro)
@@ -30,9 +30,11 @@
   <!-- Generates an Underwater Lidar model and attaches it to a parent link
        Sensor parameters align with those in the 3D at Depth SL3 datasheet -->
-  <xacro:macro name="uwl_macro" params="namespace parent_link *origin">
+  <xacro:macro name="uwl_macro" params="namespace parent_link *origin pan tilt">
     <xacro:uw_lidar_plugin_macro
       namespace="${namespace}"
       suffix=""
-      parent_link="${parent_link}" >
+      parent_link="${parent_link}"
+      pan="${pan}"
+      tilt="${tilt}" >
       <xacro:insert_block name="origin"/>
     </xacro:uw_lidar_plugin_macro>
@@ -113,5 +115,5 @@
   <!-- Generates the uw_lidar model with stand and motion control plugin -->
   <xacro:macro name="uw_lidar_plugin_macro"
-    params="namespace suffix parent_link *origin">
+    params="namespace suffix parent_link *origin pan tilt">
     <link name="${namespace}/uwl${suffix}_link">
       <inertial>
@@ -221,6 +223,6 @@
        <plugin name="pulse_lidar_control" filename="libgazebo_ros_pulse_lidar_plugin.so" >
         <robot_namespace>${namespace}</robot_namespace>
-         <pan_position>0</pan_position>
-         <tilt_position>0</tilt_position>
+         <pan_position>${pan}</pan_position>
+         <tilt_position>${tilt}</tilt_position>
        </plugin>
     </gazebo>

File: urdf/uw_lidar_pedestal_robot.xacro (robot description, xacro)
@@ -24,5 +24,5 @@
     </collision>
   </link>
-  <xacro:uwl_macro namespace="uwl" parent_link="robot_base_link">
+  <xacro:uwl_macro namespace="uwl" parent_link="robot_base_link" pan="-${pi/2}" tilt="0">
     <origin xyz="0 0 0.25" rpy="0 0 -${pi/2}"/>
   </xacro:uwl_macro>

File: urdf/uw_lidar_robot.xacro (robot description, xacro)
@@ -30,5 +30,5 @@
     <child link="robot_link"/>
   </joint>
-  <xacro:uwl_macro namespace="uwl" parent_link="robot_base_link">
+  <xacro:uwl_macro namespace="uwl" parent_link="robot_base_link" pan="0" tilt="0">
     <origin xyz="0.48 0 1.41" rpy="0 0 ${pi/2}"/>
   </xacro:uwl_macro>

Commit message: set inertial reference frame for rviz

File: urdf/uw_lidar.xacro (robot description, xacro)
@@ -30,9 +30,10 @@
   <!-- Generates an Underwater Lidar model and attaches it to a parent link
        Sensor parameters align with those in the 3D at Depth SL3 datasheet -->
-  <xacro:macro name="uwl_macro" params="namespace parent_link *origin pan tilt">
+  <xacro:macro name="uwl_macro" params="namespace parent_link *origin pan tilt inertial_reference_frame">
     <xacro:uw_lidar_plugin_macro
       namespace="${namespace}"
       suffix=""
       parent_link="${parent_link}"
+      reference_frame="${inertial_reference_frame}"
       pan="${pan}"
       tilt="${tilt}" >
@@ -41,5 +42,5 @@
   </xacro:macro>
   <!-- Generates a Lidar sensor -->
-  <xacro:macro name="uw_lidar_sensor" params="namespace suffix update_rate">
+  <xacro:macro name="uw_lidar_sensor" params="namespace suffix update_rate reference_frame">
     <link name="${namespace}/uwl${suffix}_sensor_link">
       <inertial>
@@ -62,6 +63,6 @@
        <always_on>true</always_on>
        <plugin name="pulse_lidar_sensing" filename="libgazebo_ros_velodyne_gpu_laser.so">
-           <topicName>nps_uwl/points</topicName>
-           <frameName>nps_uwl/pulse_lidar_link</frameName>
+           <topicName>nps_uwl_points</topicName>
+           <static_reference_frame>${reference_frame}</static_reference_frame>
            <min_intensity>0</min_intensity>
            <min_range>1</min_range>
@@ -115,5 +116,5 @@
   <!-- Generates the uw_lidar model with stand and motion control plugin -->
   <xacro:macro name="uw_lidar_plugin_macro"
-    params="namespace suffix parent_link *origin pan tilt">
+    params="namespace suffix parent_link *origin pan tilt reference_frame">
     <link name="${namespace}/uwl${suffix}_link">
       <inertial>
@@ -218,5 +219,5 @@
     <xacro:uw_lidar_sensor
       namespace="${namespace}" suffix=""
-      update_rate="40">
+      update_rate="40" reference_frame="${reference_frame}">
     </xacro:uw_lidar_sensor>
     <gazebo>

File: urdf/uw_lidar_pedestal_robot.xacro (robot description, xacro)
@@ -1,4 +1,5 @@
 <?xml version="1.0"?>
 <robot xmlns:xacro="http://www.ros.org/wiki/xacro" name="uw_lidar_pedestal">
+  <xacro:arg name="inertial_reference_frame" default="robot_base_link"/>
   <xacro:include filename="$(find nps_uw_sensors_gazebo)/urdf/uw_lidar.xacro"/>
   <!-- Used for fixing robot to Gazebo 'base_link' -->
@@ -24,5 +25,7 @@
     </collision>
   </link>
-  <xacro:uwl_macro namespace="uwl" parent_link="robot_base_link" pan="-${pi/2}" tilt="0">
+  <xacro:uwl_macro namespace="uwl" parent_link="robot_base_link"
+                   inertial_reference_frame="$(arg inertial_reference_frame)"
+                   pan="-${pi/2}" tilt="0">
     <origin xyz="0 0 0.25" rpy="0 0 -${pi/2}"/>
   </xacro:uwl_macro>

File: urdf/uw_lidar_robot.xacro (robot description, xacro)
@@ -1,4 +1,5 @@
 <?xml version="1.0"?>
 <robot xmlns:xacro="http://www.ros.org/wiki/xacro" name="uw_lidar">
+  <xacro:arg name="inertial_reference_frame" default="world"/>
   <xacro:include filename="$(find nps_uw_sensors_gazebo)/urdf/uw_lidar.xacro"/>
   <link name="robot_base_link"/>
@@ -30,5 +31,7 @@
     <child link="robot_link"/>
   </joint>
-  <xacro:uwl_macro namespace="uwl" parent_link="robot_base_link" pan="0" tilt="0">
+  <xacro:uwl_macro namespace="uwl" parent_link="robot_base_link"
+                   inertial_reference_frame="$(arg inertial_reference_frame)"
+                   pan="0" tilt="0">
     <origin xyz="0.48 0 1.41" rpy="0 0 ${pi/2}"/>
   </xacro:uwl_macro>
