Commit message: Created SDF models for all of the performer DVLs
Refactoring in response to Brian's input IRT PR#6.

Moved meshes into the SDF models, and modified the URDF (Xacro) files
to use those meshes rather than ones from a single "meshes" directory.

Meshes for the Teledyne WHN, Teledyne Explorer 1000, and Nortek
DVL1000-4000m are correct.  The other models (SDF and URDF) use the
closest match of the 3 meshes that we have at present.  They have
been named according to the DVL for which they're being used, so
as the actual meshes are developed they can replace what's currently
in the model-specific meshes directory and everything will work.

File: models/uuvsim_teledyne_whn_urdf/model.urdf (robot description, URDF)
Before this commit: robot teledyne_whn, 6 links, 5 joints
Links:
- link dvl_link: geometry collision cylinder length=0.2445 radius=0.1126; visual mesh filename=model://uuvsim_teledyne_whn_urdf/meshes/WorkhorseNavigator.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

File: urdf/uuvsim_nortek_dvl1000_300.xacro (robot description, xacro)
@@ -126,5 +126,5 @@
       <visual>
         <geometry>
-          <mesh filename="package://nps_uw_sensors_gazebo/meshes/DVL1000-4000m.dae"/>
+          <mesh filename="package://nps_uw_sensors_gazebo/models/whoi_nortek_dvl1000_300/meshes/DVL1000-300m.dae"/>
         </geometry>
         <origin xyz="0 0 0" rpy="0 -1.5707963267948966 0"/>

File: urdf/uuvsim_nortek_dvl1000_4000.xacro (robot description, xacro)
@@ -126,5 +126,5 @@
       <visual>
         <geometry>
-          <mesh filename="package://nps_uw_sensors_gazebo/meshes/DVL1000-4000m.dae"/>
+          <mesh filename="package://nps_uw_sensors_gazebo/models/whoi_nortek_dvl1000_4000/meshes/DVL1000-4000m.dae"/>
         </geometry>
         <origin xyz="0 0 0" rpy="0 -1.5707963267948966 0"/>

File: urdf/uuvsim_nortek_dvl500_300.xacro (robot description, xacro)
@@ -127,5 +127,5 @@
         <geometry>
           <!-- Replace with Nortek DVL500 mesh when available -->
-          <mesh filename="package://nps_uw_sensors_gazebo/meshes/DVL1000-4000m.dae"/>
+          <mesh filename="package://nps_uw_sensors_gazebo/models/whoi_nortek_dvl500_300/meshes/DVL500-300m.dae"/>
         </geometry>
         <origin xyz="0 0 0" rpy="0 -1.5707963267948966 0"/>

File: urdf/uuvsim_nortek_dvl500_6000.xacro (robot description, xacro)
@@ -127,5 +127,5 @@
         <geometry>
           <!-- Replace with Nortek DVL500 mesh when available -->
-          <mesh filename="package://nps_uw_sensors_gazebo/meshes/DVL1000-4000m.dae"/>
+          <mesh filename="package://nps_uw_sensors_gazebo/models/whoi_nortek_dvl500_6000/meshes/DVL500-6000m.dae"/>
         </geometry>
         <origin xyz="0 0 0" rpy="0 -1.5707963267948966 0"/>

File: urdf/uuvsim_sonardyne_syrinx600.xacro (robot description, xacro)
@@ -127,7 +127,7 @@
         <geometry>
           <!-- Replace with Sonardyne Syrinx 600 mesh when available -->
-          <mesh filename="package://nps_uw_sensors_gazebo/meshes/WorkhorseNavigator.dae"/>
+          <mesh filename="package://nps_uw_sensors_gazebo/models/whoi_sonardyne_syrinx600/meshes/Syrinx600.dae"/>
         </geometry>
-        <origin xyz="0 0 0" rpy="0 1.5707963267948966 0"/>
+        <origin xyz="0 0 0" rpy="0 3.141592653589793 0"/>
       </visual>
       <collision>

File: urdf/uuvsim_teledyne_explorer_1000.xacro (robot description, xacro)
@@ -128,5 +128,5 @@
       <visual>
         <geometry>
-          <mesh filename="package://nps_uw_sensors_gazebo/meshes/TeledyneMarineExplorer.dae"/>
+          <mesh filename="package://nps_uw_sensors_gazebo/models/whoi_teledyne_explorer1000/meshes/MarineExplorer.dae"/>
         </geometry>
         <origin xyz="0 0 0" rpy="0 0 1.5707963267948966"/>

File: urdf/uuvsim_teledyne_explorer_4000.xacro (robot description, xacro)
@@ -127,5 +127,5 @@
       <visual>
         <geometry>
-          <mesh filename="package://nps_uw_sensors_gazebo/meshes/TeledyneMarineExplorer.dae"/>
+          <mesh filename="package://nps_uw_sensors_gazebo/models/whoi_teledyne_explorer4000/meshes/MarineExplorer.dae"/>
         </geometry>
         <origin xyz="0 0 0" rpy="0 0 1.5707963267948966"/>

File: urdf/uuvsim_teledyne_whn.xacro (robot description, xacro)
@@ -126,5 +126,5 @@
       <visual>
         <geometry>
-          <mesh filename="package://nps_uw_sensors_gazebo/meshes/WorkhorseNavigator.dae"/>
+          <mesh filename="package://nps_uw_sensors_gazebo/models/whoi_teledyne_whn/meshes/WorkhorseNavigator.dae"/>
         </geometry>
         <origin xyz="0 0 0" rpy="0 1.5707963267948966 0"/>

File: urdf/whoi_nortek_dvl1000_300.xacro (robot description, xacro)
@@ -44,5 +44,6 @@
       <visual>
         <geometry>
-          <mesh filename="package://nps_uw_sensors_gazebo/meshes/DVL1000-4000m.dae"/>
+<!--          <mesh filename="$(find nps_uw_sensors_gazebo)/models/whoi_nortek_dvl1000_300/meshes/DVL1000-300m.dae"/> -->
+          <mesh filename="package://nps_uw_sensors_gazebo/models/whoi_nortek_dvl1000_300/meshes/DVL1000-300m.dae"/>
         </geometry>
         <origin xyz="${xyz}" rpy="0 ${pi} 0"/>

File: urdf/whoi_nortek_dvl1000_4000.xacro (robot description, xacro)
@@ -44,5 +44,5 @@
       <visual>
         <geometry>
-          <mesh filename="package://nps_uw_sensors_gazebo/meshes/DVL1000-4000m.dae"/>
+          <mesh filename="package://nps_uw_sensors_gazebo/models/whoi_nortek_dvl1000_4000/meshes/DVL1000-4000m.dae"/>
         </geometry>
         <origin xyz="${xyz}" rpy="0 ${pi} 0"/>

File: urdf/whoi_nortek_dvl500_300.xacro (robot description, xacro)
@@ -45,5 +45,5 @@
         <geometry>
           <!-- Replace mesh with correct one once it's available -->
-          <mesh filename="package://nps_uw_sensors_gazebo/meshes/DVL1000-4000m.dae"/>
+          <mesh filename="package://nps_uw_sensors_gazebo/models/whoi_nortek_dvl500_300/meshes/DVL500-300m.dae"/>
         </geometry>
         <origin xyz="${xyz}" rpy="0 ${pi} 0"/>

File: urdf/whoi_nortek_dvl500_6000.xacro (robot description, xacro)
@@ -45,5 +45,5 @@
         <geometry>
           <!-- Replace mesh with correct one once it's available -->
-          <mesh filename="package://nps_uw_sensors_gazebo/meshes/DVL1000-4000m.dae"/>
+          <mesh filename="package://nps_uw_sensors_gazebo/models/whoi_nortek_dvl500_6000/meshes/DVL500-6000m.dae"/>
         </geometry>
         <origin xyz="${xyz}" rpy="0 ${pi} 0"/>

File: urdf/whoi_sonardyne_syrinx600.xacro (robot description, xacro)
@@ -45,7 +45,7 @@
         <geometry>
           <!-- Replace mesh with correct one once it's available -->
-          <mesh filename="package://nps_uw_sensors_gazebo/meshes/WorkhorseNavigator.dae"/>
+          <mesh filename="package://nps_uw_sensors_gazebo/models/whoi_sonardyne_syrinx600/meshes/Syrinx600.dae"/>
         </geometry>
-        <origin xyz="${xyz}" rpy="0 0 0"/>
+        <origin xyz="${xyz}" rpy="0 ${pi} 0"/>
       </visual>
       <collision>

File: urdf/whoi_teledyne_explorer_1000.xacro (robot description, xacro)
@@ -45,5 +45,5 @@
       <visual>
         <geometry>
-          <mesh filename="package://nps_uw_sensors_gazebo/meshes/TeledyneMarineExplorer.dae"/>
+          <mesh filename="package://nps_uw_sensors_gazebo/models/whoi_teledyne_explorer1000/meshes/MarineExplorer.dae"/>
         </geometry>
         <origin xyz="${xyz}" rpy="${-0.5*pi} 0 ${-0.5*pi}"/>

File: urdf/whoi_teledyne_explorer_4000.xacro (robot description, xacro)
@@ -45,5 +45,5 @@
       <visual>
         <geometry>
-          <mesh filename="package://nps_uw_sensors_gazebo/meshes/TeledyneMarineExplorer.dae"/>
+          <mesh filename="package://nps_uw_sensors_gazebo/models/whoi_teledyne_explorer4000/meshes/MarineExplorer.dae"/>
         </geometry>
         <origin xyz="${xyz}" rpy="${-0.5*pi} 0 ${-0.5*pi}"/>

File: urdf/whoi_teledyne_whn.xacro (robot description, xacro)
@@ -44,5 +44,5 @@
       <visual>
         <geometry>
-          <mesh filename="package://nps_uw_sensors_gazebo/meshes/WorkhorseNavigator.dae"/>
+          <mesh filename="package://nps_uw_sensors_gazebo/models/whoi_teledyne_whn/meshes/WorkhorseNavigator.dae"/>
         </geometry>
         <origin xyz="${xyz}" rpy="0 0 0"/>

File: urdf/whoi_teledyne_whn_robot.xacro (robot description, xacro)
@@ -2,5 +2,4 @@
 <robot xmlns:xacro="http://www.ros.org/wiki/xacro" name="teledyne_whn">
   <xacro:include filename="$(find nps_uw_sensors_gazebo)/urdf/whoi_teledyne_whn.xacro"/>
-  <!-- Simple example "UUV" (really it's just a cylinder) -->
   <link name="robot_base_link"/>
   <link name="robot_link">
